Commit message: gz ok little drift

File: dshape_description/urdf/dshape_core.xacro (robot description, xacro)
@@ -29,5 +29,5 @@
       <geometry>
         <mesh
-          filename="dshape_description/meshes/base_link.STL" />
+          filename="package://dshape_description/meshes/base_link.STL" />
       </geometry>
       <material
@@ -43,5 +43,5 @@
       <geometry>
         <mesh
-          filename="dshape_description/meshes/base_link.STL" />
+          filename="package://dshape_description/meshes/base_link.STL" />
       </geometry>
     </collision>
@@ -69,5 +69,5 @@
       <geometry>
         <mesh
-          filename="dshape_description/meshes/right_wheel.STL" />
+          filename="package://dshape_description/meshes/right_wheel.STL" />
       </geometry>
       <material
@@ -83,6 +83,17 @@
       <geometry>
         <mesh
-          filename="dshape_description/meshes/right_wheel.STL" />
-      </geometry>
+          filename="package://dshape_description/meshes/right_wheel.STL" />
+      </geometry>
+      <surface>
+            <friction>
+                <ode>
+                    <mu>1</mu>
+                    <mu2>1</mu2>
+                    <fdir1>0 0 0</fdir1>
+                    <slip1>0</slip1>
+                    <slip2>0</slip2>
+                </ode>
+            </friction>
+        </surface>
     </collision>
   </link>
@@ -122,5 +133,5 @@
       <geometry>
         <mesh
-          filename="dshape_description/meshes/left_wheel.STL" />
+          filename="package://dshape_description/meshes/left_wheel.STL" />
       </geometry>
       <material
@@ -136,6 +147,17 @@
       <geometry>
         <mesh
-          filename="dshape_description/meshes/left_wheel.STL" />
-      </geometry>
+          filename="package://dshape_description/meshes/left_wheel.STL" />
+      </geometry>
+      <surface>
+            <friction>
+                <ode>
+                    <mu>1</mu>
+                    <mu2>1</mu2>
+                    <fdir1>0 0 0</fdir1>
+                    <slip1>0</slip1>
+                    <slip2>0</slip2>
+                </ode>
+            </friction>
+        </surface>
     </collision>
   </link>
@@ -172,7 +194,11 @@
   <gazebo reference="right_wheel">
     <material>Gazebo/Yellow</material>
+    <mu1>1.0</mu1>
+    <mu2>1.0</mu2>
   </gazebo>
    <gazebo reference="left_wheel">
     <material>Gazebo/Yellow</material>
+    <mu1>1.0</mu1>
+    <mu2>1.0</mu2>
   </gazebo>
    <gazebo reference="lidar">

File: dshape_description/urdf/urdf.urdf (robot description, URDF)
Before this commit: robot dshape, 7 links, 6 joints
Links:
- link base_link: geometry collision mesh filename=/home/mr_robot/ros2/developer_ws/src/dshape/dshape_descript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; visual mesh filename=/home/mr_robot/ros2/developer_ws/src/dshape/dshape_descript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
- link left_wheel: geometry collision mesh filename=/home/mr_robot/ros2/developer_ws/src/dshape/dshape_descript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; visual mesh filename=/home/mr_robot/ros2/developer_ws/src/dshape/dshape_descript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
- link right_wheel: geometry collision mesh filename=/home/mr_robot/ros2/developer_ws/src/dshape/dshape_descript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; visual mesh filename=/home/mr_robot/ros2/developer_ws/src/dshape/dshape_descript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
Joints:
- joint camera_joint: origin xyz=0 0 0.3 rpy=0 0 0 -> xyz=0 0 0.03 rpy=0 0 0
- joint lidar_joint: origin xyz=0 0 0.2 rpy=0 0 0 -> xyz=0 0 0.02 rpy=0 0 0
