Commit message: cm error

File: dshape_description/urdf/robot.urdf.xacro (robot description, xacro)
@@ -1,7 +1,7 @@
 <?xml version="1.0"?>
 <robot xmlns:xacro="http://www.ros.org/wiki/xacro"  name="dshape">
+    <xacro:arg name="prefix" default="" />
     <xacro:include filename="dshape_core.xacro" />
-    <xacro:include filename="lidar.xacro" />
     <xacro:include filename="ros2_control.xacro" />
-    <xacro:include filename="camera.xacro" />
+    <xacro:diffbot_ros2_control name="DiffBot" prefix="$(arg prefix)" />
 </robot>

File: dshape_description/urdf/ros2_control.xacro (robot description, xacro)
@@ -1,37 +1,33 @@
 <?xml version="1.0"?>
 <robot xmlns:xacro="http://www.ros.org/wiki/xacro">
-    <ros2_control name="GazeboSystem" type="system">
-        <hardware>
-            <plugin>gazebo_ros2_control/GazeboSystem</plugin>
-        </hardware>
-        <joint name="left_wheel_joint">
-            <command_interface name="velocity">
-                <param name="min">-10</param>
-                <param name="max">10</param>
-            </command_interface>
-            <state_interface name="velocity"/>
-            <state_interface name="position"/>
-        </joint>
-        <joint name="right_wheel_joint">
-            <command_interface name="velocity">
-                <param name="min">-10</param>
-                <param name="max">10</param>
-            </command_interface>
-            <state_interface name="velocity"/>
-            <state_interface name="position"/>
-        </joint>
-    </ros2_control>
-    <gazebo>
-        <plugin name="gazebo_ros2_control" filename="libgazebo_ros2_control.so">
-            <robot_param>robot_description</robot_param>
-            <robot_param_node>robot_state_publisher</robot_param_node>
-            <parameters>$(find dshape_description)/config/my_controllers.yaml</parameters>
-            <!-- Output -->
-            <odometry_frame>odom</odometry_frame>
-            <robot_base_frame>base_footprint</robot_base_frame>
-            <publish_odom>true</publish_odom>
-            <publish_odom_tf>true</publish_odom_tf>
-            <publish_wheel_tf>true</publish_wheel_tf>
-        </plugin>
-    </gazebo>
+    <xacro:macro name="diffbot_ros2_control" params="name prefix">
+        <ros2_control name="${name}" type="system">
+            <hardware>
+                <plugin>diffdrive_stm32/DiffDriveStm32Hardware</plugin>
+                <param name="left_wheel_name">left_wheel_joint</param>
+                <param name="right_wheel_name">right_wheel_joint</param>
+                <param name="loop_rate" >50</param>
+                <param name="device">/dev/ttyUSB0</param><!--fixed-->
+                <param name="baud_rate">115200</param>
+                <param name="timeout_ms">1000</param>
+                <param name="enc_counts_per_rev">1320</param>
+            </hardware>
+            <joint name="left_wheel_joint">
+                <command_interface name="velocity">
+                    <param name="min">-50</param>
+                    <param name="max">50</param>
+                </command_interface>
+                <state_interface name="velocity"/>
+                <state_interface name="position"/>
+            </joint>
+            <joint name="right_wheel_joint">
+                <command_interface name="velocity">
+                    <param name="min">-50</param>
+                    <param name="max">50</param>
+                </command_interface>
+                <state_interface name="velocity"/>
+                <state_interface name="position"/>
+            </joint>
+        </ros2_control>
+    </xacro:macro>
 </robot>

File: dshape_description/urdf/urdf.urdf (robot description, URDF)
Before this commit: robot dshape, 7 links, 6 joints
Links:
- removed link camera_link_optical
- link base_link: geometry collision mesh filename=package://dshape_description/meshes/base_link.STL; visual mesh filename=package://dshape_description/meshes/base_link.STL
- link left_wheel: geometry collision mesh filename=package://dshape_description/meshes/left_wheel.STL; visual mesh filename=package://dshape_description/meshes/left_wheel.STL
- link right_wheel: geometry collision mesh filename=package://dshape_description/meshes/right_wheel.STL; visual mesh filename=package://dshape_description/meshes/right_wheel.STL
Joints:
- removed joint camera_optical_joint
